File: Adapter-IO4-test_array.brd (EAGLE design)
At the start: 128.3 x 106.7 mm, 89 parts

Commit message: simplified design
Parts:
- removed LED5X11, LED5X12, LED5X21, LED5X22, LED6X11, LED6X12, LED6X21, LED6X22, LED7X11, LED7X12, LED7X21, LED7X22, LED8X11, LED8X12, LED8X21, LED8X22: (no value), SPCoast:LED5MM
- removed SW4X1: (no value), SPCoast:BOARD-10X10-2X2-PANEL
- moved Q1X22 36.7 mm to (55.7, 91.3), turned to 90 degrees
- moved Q2X22 36.7 mm to (65.9, 91.3), turned to 90 degrees
- moved Q3X22 36.7 mm to (76.0, 91.3), turned to 90 degrees
- moved Q4X22 36.7 mm to (86.2, 91.3), turned to 90 degrees
- moved Q1X12 36.7 mm to (5.71, 91.3), turned to 90 degrees
- moved Q2X12 36.7 mm to (15.9, 91.3), turned to 90 degrees
- moved Q3X12 36.7 mm to (26.0, 91.3), turned to 90 degrees
- moved Q4X12 36.7 mm to (36.2, 91.3), turned to 90 degrees
- moved Q1X21 29.2 mm to (55.7, 41.3), turned to 90 degrees
- moved Q2X21 29.2 mm to (65.9, 41.3), turned to 90 degrees
- moved Q3X21 29.2 mm to (76.0, 41.3), turned to 90 degrees
- moved Q4X21 29.2 mm to (86.2, 41.3), turned to 90 degrees
- moved Q1X11 29.2 mm to (5.71, 41.3), turned to 90 degrees
- moved Q2X11 29.2 mm to (15.9, 41.3), turned to 90 degrees
- moved Q3X11 29.2 mm to (26.0, 41.3), turned to 90 degrees
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Connections:
- net GNDX11: no longer LED5X11.K, LED6X11.K, LED7X11.K, LED8X11.K
- net GNDX12: no longer LED5X12.K, LED6X12.K, LED7X12.K, LED8X12.K
- net GNDX21: no longer LED5X21.K, LED6X21.K, LED7X21.K, LED8X21.K
- net GNDX22: no longer LED5X22.K, LED6X22.K, LED7X22.K, LED8X22.K
- net N$16X11: no longer LED8X11.A
- net N$16X12: no longer LED8X12.A
- net N$16X21: no longer LED8X21.A
- net N$16X22: no longer LED8X22.A
- net N$2X11: no longer LED5X11.A
- net N$2X12: no longer LED5X12.A
- net N$2X21: no longer LED5X21.A
- net N$2X22: no longer LED5X22.A
- net N$4X11: no longer LED6X11.A
- net N$4X12: no longer LED6X12.A
- net N$4X21: no longer LED6X21.A
- net N$4X22: no longer LED6X22.A
- net N$6X11: no longer LED7X11.A
- net N$6X12: no longer LED7X12.A
- net N$6X21: no longer LED7X21.A
- net N$6X22: no longer LED7X22.A
Routing:
- net N$7X22: track 95.0 -> 70.2 mm
- net N$7X21: track 95.0 -> 70.2 mm
- net N$7X12: track 95.0 -> 70.2 mm
- net N$7X11: track 95.0 -> 70.2 mm
- net N$10X11: track 75.1 -> 59.5 mm
- net N$10X12: track 75.1 -> 59.5 mm
- net N$10X22: track 75.1 -> 59.5 mm
- net N$10X21: track 75.1 -> 59.5 mm
- net N$8X21: track 76.7 -> 63.1 mm, vias 3 -> 2
- net N$8X12: track 76.7 -> 63.1 mm, vias 3 -> 2
- net N$8X22: track 76.7 -> 63.1 mm, vias 3 -> 2
- net N$8X11: track 76.7 -> 63.1 mm, vias 3 -> 2
- net N$9X21: track 76.5 -> 63.4 mm, vias 3 -> 2
- net N$9X22: track 76.5 -> 63.4 mm, vias 3 -> 2
- net N$9X11: track 76.5 -> 63.4 mm, vias 3 -> 2
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Other:
- board size 128.3 x 106.7 mm -> 107.6 x 107.6 mm
- board text added: "2020-05"
- board text added: "V-Score"
- board text added: "v1.1"
- board text removed: "2020-01"
- board text removed: "v1.0"

Commit message: added value G to LEDs
Parts:
- LED1X11, LED1X12, LED1X21, LED1X22, LED2X11, LED2X12, LED2X21, LED2X22, LED3X11, LED3X12, LED3X21, LED3X22, LED4X11, LED4X12, LED4X21, LED4X22: value (none) -> G
Changed lines of the file:
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@@
 <element name="CON1X11" library="SPCoast" package="RJ25-INVERTED" value="" x="4.445" y="15.875" rot="R270"/>
 <element name="CON2X11" library="SPCoast" package="1X06_LOCK" value="" x="45.085" y="10.16" rot="R90"/>
-<element name="LED1X11" library="SPCoast" package="0805-LED" value="" x="10.795" y="37.465"/>
-<element name="LED2X11" library="SPCoast" package="0805-LED" value="" x="20.955" y="37.465"/>
-<element name="LED3X11" library="SPCoast" package="0805-LED" value="" x="31.115" y="37.465"/>
-<element name="LED4X11" library="SPCoast" package="0805-LED" value="" x="41.275" y="37.465"/>
+<element name="LED1X11" library="SPCoast" package="0805-LED" value="G" x="10.795" y="37.465"/>
+<element name="LED2X11" library="SPCoast" package="0805-LED" value="G" x="20.955" y="37.465"/>
+<element name="LED3X11" library="SPCoast" package="0805-LED" value="G" x="31.115" y="37.465"/>
+<element name="LED4X11" library="SPCoast" package="0805-LED" value="G" x="41.275" y="37.465"/>
 <element name="Q1X11" library="SPCoast" package="SOT23-3" value="" x="5.715" y="41.275" rot="R90"/>
 <element name="Q2X11" library="SPCoast" package="SOT23-3" value="" x="15.875" y="41.275" rot="R90"/>
@@
 <element name="CON1X12" library="SPCoast" package="RJ25-INVERTED" value="" x="4.445" y="65.875" rot="R270"/>
 <element name="CON2X12" library="SPCoast" package="1X06_LOCK" value="" x="45.085" y="60.16" rot="R90"/>
-<element name="LED1X12" library="SPCoast" package="0805-LED" value="" x="10.795" y="87.465"/>
-<element name="LED2X12" library="SPCoast" package="0805-LED" value="" x="20.955" y="87.465"/>
-<element name="LED3X12" library="SPCoast" package="0805-LED" value="" x="31.115" y="87.465"/>
-<element name="LED4X12" library="SPCoast" package="0805-LED" value="" x="41.275" y="87.465"/>
+<element name="LED1X12" library="SPCoast" package="0805-LED" value="G" x="10.795" y="87.465"/>
+<element name="LED2X12" library="SPCoast" package="0805-LED" value="G" x="20.955" y="87.465"/>
+<element name="LED3X12" library="SPCoast" package="0805-LED" value="G" x="31.115" y="87.465"/>
+<element name="LED4X12" library="SPCoast" package="0805-LED" value="G" x="41.275" y="87.465"/>
 <element name="Q1X12" library="SPCoast" package="SOT23-3" value="" x="5.715" y="91.275" rot="R90"/>
 <element name="Q2X12" library="SPCoast" package="SOT23-3" value="" x="15.875" y="91.275" rot="R90"/>
@@
 <element name="CON1X21" library="SPCoast" package="RJ25-INVERTED" value="" x="54.445" y="15.875" rot="R270"/>
 <element name="CON2X21" library="SPCoast" package="1X06_LOCK" value="" x="95.085" y="10.16" rot="R90"/>
-<element name="LED1X21" library="SPCoast" package="0805-LED" value="" x="60.795" y="37.465"/>
-<element name="LED2X21" library="SPCoast" package="0805-LED" value="" x="70.955" y="37.465"/>
-<element name="LED3X21" library="SPCoast" package="0805-LED" value="" x="81.115" y="37.465"/>
-<element name="LED4X21" library="SPCoast" package="0805-LED" value="" x="91.275" y="37.465"/>
+<element name="LED1X21" library="SPCoast" package="0805-LED" value="G" x="60.795" y="37.465"/>
+<element name="LED2X21" library="SPCoast" package="0805-LED" value="G" x="70.955" y="37.465"/>
+<element name="LED3X21" library="SPCoast" package="0805-LED" value="G" x="81.115" y="37.465"/>
+<element name="LED4X21" library="SPCoast" package="0805-LED" value="G" x="91.275" y="37.465"/>
 <element name="Q1X21" library="SPCoast" package="SOT23-3" value="" x="55.715" y="41.275" rot="R90"/>
 <element name="Q2X21" library="SPCoast" package="SOT23-3" value="" x="65.875" y="41.275" rot="R90"/>
@@
 <element name="CON1X22" library="SPCoast" package="RJ25-INVERTED" value="" x="54.445" y="65.875" rot="R270"/>
 <element name="CON2X22" library="SPCoast" package="1X06_LOCK" value="" x="95.085" y="60.16" rot="R90"/>
-<element name="LED1X22" library="SPCoast" package="0805-LED" value="" x="60.795" y="87.465"/>
-<element name="LED2X22" library="SPCoast" package="0805-LED" value="" x="70.955" y="87.465"/>
-<element name="LED3X22" library="SPCoast" package="0805-LED" value="" x="81.115" y="87.465"/>
-<element name="LED4X22" library="SPCoast" package="0805-LED" value="" x="91.275" y="87.465"/>
+<element name="LED1X22" library="SPCoast" package="0805-LED" value="G" x="60.795" y="87.465"/>
+<element name="LED2X22" library="SPCoast" package="0805-LED" value="G" x="70.955" y="87.465"/>
+<element name="LED3X22" library="SPCoast" package="0805-LED" value="G" x="81.115" y="87.465"/>
+<element name="LED4X22" library="SPCoast" package="0805-LED" value="G" x="91.275" y="87.465"/>
 <element name="Q1X22" library="SPCoast" package="SOT23-3" value="" x="55.715" y="91.275" rot="R90"/>
 <element name="Q2X22" library="SPCoast" package="SOT23-3" value="" x="65.875" y="91.275" rot="R90"/>

Commit message: array needed R and Q values as well
Parts:
- Q1X11, Q1X12, Q1X21, Q1X22, Q2X11, Q2X12, Q2X21, Q2X22, Q3X11, Q3X12, Q3X21, Q3X22, Q4X11, Q4X12, Q4X21, Q4X22: value (none) -> p-fet
- R1X11, R1X12, R1X21, R1X22, R2X11, R2X12, R2X21, R2X22, R3X11, R3X12, R3X21, R3X22, R4X11, R4X12, R4X21, R4X22: value (none) -> 2k0
Changed lines of the file:
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@@
 <element name="LED3X11" library="SPCoast" package="0805-LED" value="G" x="31.115" y="37.465"/>
 <element name="LED4X11" library="SPCoast" package="0805-LED" value="G" x="41.275" y="37.465"/>
-<element name="Q1X11" library="SPCoast" package="SOT23-3" value="" x="5.715" y="41.275" rot="R90"/>
-<element name="Q2X11" library="SPCoast" package="SOT23-3" value="" x="15.875" y="41.275" rot="R90"/>
-<element name="Q3X11" library="SPCoast" package="SOT23-3" value="" x="26.035" y="41.275" rot="R90"/>
-<element name="Q4X11" library="SPCoast" package="SOT23-3" value="" x="36.195" y="41.275" rot="R90"/>
-<element name="R1X11" library="SPCoast" package="0805-RES" value="" x="5.715" y="37.465" rot="R180"/>
-<element name="R2X11" library="SPCoast" package="0805-RES" value="" x="15.875" y="37.465" rot="R180"/>
-<element name="R3X11" library="SPCoast" package="0805-RES" value="" x="26.035" y="37.465" rot="R180"/>
-<element name="R4X11" library="SPCoast" package="0805-RES" value="" x="36.195" y="37.465" rot="R180"/>
+<element name="Q1X11" library="SPCoast" package="SOT23-3" value="p-fet" x="5.715" y="41.275" rot="R90"/>
+<element name="Q2X11" library="SPCoast" package="SOT23-3" value="p-fet" x="15.875" y="41.275" rot="R90"/>
+<element name="Q3X11" library="SPCoast" package="SOT23-3" value="p-fet" x="26.035" y="41.275" rot="R90"/>
+<element name="Q4X11" library="SPCoast" package="SOT23-3" value="p-fet" x="36.195" y="41.275" rot="R90"/>
+<element name="R1X11" library="SPCoast" package="0805-RES" value="2k0" x="5.715" y="37.465" rot="R180"/>
+<element name="R2X11" library="SPCoast" package="0805-RES" value="2k0" x="15.875" y="37.465" rot="R180"/>
+<element name="R3X11" library="SPCoast" package="0805-RES" value="2k0" x="26.035" y="37.465" rot="R180"/>
+<element name="R4X11" library="SPCoast" package="0805-RES" value="2k0" x="36.195" y="37.465" rot="R180"/>
 <element name="SW1X11" library="SPCoast" package="B3F-10XX" value="" x="10.795" y="29.845" rot="R90"/>
 <element name="SW2X11" library="SPCoast" package="B3F-10XX" value="" x="20.955" y="29.845" rot="R90"/>
@@
 <element name="LED3X12" library="SPCoast" package="0805-LED" value="G" x="31.115" y="87.465"/>
 <element name="LED4X12" library="SPCoast" package="0805-LED" value="G" x="41.275" y="87.465"/>
-<element name="Q1X12" library="SPCoast" package="SOT23-3" value="" x="5.715" y="91.275" rot="R90"/>
-<element name="Q2X12" library="SPCoast" package="SOT23-3" value="" x="15.875" y="91.275" rot="R90"/>
-<element name="Q3X12" library="SPCoast" package="SOT23-3" value="" x="26.035" y="91.275" rot="R90"/>
-<element name="Q4X12" library="SPCoast" package="SOT23-3" value="" x="36.195" y="91.275" rot="R90"/>
-<element name="R1X12" library="SPCoast" package="0805-RES" value="" x="5.715" y="87.465" rot="R180"/>
-<element name="R2X12" library="SPCoast" package="0805-RES" value="" x="15.875" y="87.465" rot="R180"/>
-<element name="R3X12" library="SPCoast" package="0805-RES" value="" x="26.035" y="87.465" rot="R180"/>
-<element name="R4X12" library="SPCoast" package="0805-RES" value="" x="36.195" y="87.465" rot="R180"/>
+<element name="Q1X12" library="SPCoast" package="SOT23-3" value="p-fet" x="5.715" y="91.275" rot="R90"/>
+<element name="Q2X12" library="SPCoast" package="SOT23-3" value="p-fet" x="15.875" y="91.275" rot="R90"/>
+<element name="Q3X12" library="SPCoast" package="SOT23-3" value="p-fet" x="26.035" y="91.275" rot="R90"/>
+<element name="Q4X12" library="SPCoast" package="SOT23-3" value="p-fet" x="36.195" y="91.275" rot="R90"/>
+<element name="R1X12" library="SPCoast" package="0805-RES" value="2k0" x="5.715" y="87.465" rot="R180"/>
+<element name="R2X12" library="SPCoast" package="0805-RES" value="2k0" x="15.875" y="87.465" rot="R180"/>
+<element name="R3X12" library="SPCoast" package="0805-RES" value="2k0" x="26.035" y="87.465" rot="R180"/>
+<element name="R4X12" library="SPCoast" package="0805-RES" value="2k0" x="36.195" y="87.465" rot="R180"/>
 <element name="SW1X12" library="SPCoast" package="B3F-10XX" value="" x="10.795" y="79.845" rot="R90"/>
 <element name="SW2X12" library="SPCoast" package="B3F-10XX" value="" x="20.955" y="79.845" rot="R90"/>
@@
 <element name="LED3X21" library="SPCoast" package="0805-LED" value="G" x="81.115" y="37.465"/>
 <element name="LED4X21" library="SPCoast" package="0805-LED" value="G" x="91.275" y="37.465"/>
-<element name="Q1X21" library="SPCoast" package="SOT23-3" value="" x="55.715" y="41.275" rot="R90"/>
-<element name="Q2X21" library="SPCoast" package="SOT23-3" value="" x="65.875" y="41.275" rot="R90"/>
-<element name="Q3X21" library="SPCoast" package="SOT23-3" value="" x="76.035" y="41.275" rot="R90"/>
-<element name="Q4X21" library="SPCoast" package="SOT23-3" value="" x="86.195" y="41.275" rot="R90"/>
-<element name="R1X21" library="SPCoast" package="0805-RES" value="" x="55.715" y="37.465" rot="R180"/>
-<element name="R2X21" library="SPCoast" package="0805-RES" value="" x="65.875" y="37.465" rot="R180"/>
-<element name="R3X21" library="SPCoast" package="0805-RES" value="" x="76.035" y="37.465" rot="R180"/>
-<element name="R4X21" library="SPCoast" package="0805-RES" value="" x="86.195" y="37.465" rot="R180"/>
+<element name="Q1X21" library="SPCoast" package="SOT23-3" value="p-fet" x="55.715" y="41.275" rot="R90"/>
+<element name="Q2X21" library="SPCoast" package="SOT23-3" value="p-fet" x="65.875" y="41.275" rot="R90"/>
+<element name="Q3X21" library="SPCoast" package="SOT23-3" value="p-fet" x="76.035" y="41.275" rot="R90"/>
+<element name="Q4X21" library="SPCoast" package="SOT23-3" value="p-fet" x="86.195" y="41.275" rot="R90"/>
+<element name="R1X21" library="SPCoast" package="0805-RES" value="2k0" x="55.715" y="37.465" rot="R180"/>
+<element name="R2X21" library="SPCoast" package="0805-RES" value="2k0" x="65.875" y="37.465" rot="R180"/>
+<element name="R3X21" library="SPCoast" package="0805-RES" value="2k0" x="76.035" y="37.465" rot="R180"/>
+<element name="R4X21" library="SPCoast" package="0805-RES" value="2k0" x="86.195" y="37.465" rot="R180"/>
 <element name="SW1X21" library="SPCoast" package="B3F-10XX" value="" x="60.795" y="29.845" rot="R90"/>
 <element name="SW2X21" library="SPCoast" package="B3F-10XX" value="" x="70.955" y="29.845" rot="R90"/>
@@
 <element name="LED3X22" library="SPCoast" package="0805-LED" value="G" x="81.115" y="87.465"/>
 <element name="LED4X22" library="SPCoast" package="0805-LED" value="G" x="91.275" y="87.465"/>
-<element name="Q1X22" library="SPCoast" package="SOT23-3" value="" x="55.715" y="91.275" rot="R90"/>
-<element name="Q2X22" library="SPCoast" package="SOT23-3" value="" x="65.875" y="91.275" rot="R90"/>
-<element name="Q3X22" library="SPCoast" package="SOT23-3" value="" x="76.035" y="91.275" rot="R90"/>
-<element name="Q4X22" library="SPCoast" package="SOT23-3" value="" x="86.195" y="91.275" rot="R90"/>
-<element name="R1X22" library="SPCoast" package="0805-RES" value="" x="55.715" y="87.465" rot="R180"/>
-<element name="R2X22" library="SPCoast" package="0805-RES" value="" x="65.875" y="87.465" rot="R180"/>
-<element name="R3X22" library="SPCoast" package="0805-RES" value="" x="76.035" y="87.465" rot="R180"/>
-<element name="R4X22" library="SPCoast" package="0805-RES" value="" x="86.195" y="87.465" rot="R180"/>
+<element name="Q1X22" library="SPCoast" package="SOT23-3" value="p-fet" x="55.715" y="91.275" rot="R90"/>
+<element name="Q2X22" library="SPCoast" package="SOT23-3" value="p-fet" x="65.875" y="91.275" rot="R90"/>
+<element name="Q3X22" library="SPCoast" package="SOT23-3" value="p-fet" x="76.035" y="91.275" rot="R90"/>
+<element name="Q4X22" library="SPCoast" package="SOT23-3" value="p-fet" x="86.195" y="91.275" rot="R90"/>
+<element name="R1X22" library="SPCoast" package="0805-RES" value="2k0" x="55.715" y="87.465" rot="R180"/>
+<element name="R2X22" library="SPCoast" package="0805-RES" value="2k0" x="65.875" y="87.465" rot="R180"/>
+<element name="R3X22" library="SPCoast" package="0805-RES" value="2k0" x="76.035" y="87.465" rot="R180"/>
+<element name="R4X22" library="SPCoast" package="0805-RES" value="2k0" x="86.195" y="87.465" rot="R180"/>
 <element name="SW1X22" library="SPCoast" package="B3F-10XX" value="" x="60.795" y="79.845" rot="R90"/>
 <element name="SW2X22" library="SPCoast" package="B3F-10XX" value="" x="70.955" y="79.845" rot="R90"/>
